File: analog.sch (KiCad schematic (older format))
At the start: 57 parts

Commit message: [sch] use an off-the-shelf pyboard to handle the digital part
Parts:
- gave numbers to parts that had none: 55

Commit message: [pcb] layout rev1
Parts:
- removed C10, C19, C26, C5: 100nF, symbol C
- removed R14, R7: R_Variable, symbol R_Variable
- added J10, J11, J12, J13, J14, J15, J16, J17, J18, J7, J8, J9: TEST_1P, Pin_Headers:Pin_Header_Straight_1x01_Pitch2.54mm, symbol TEST_1P
- added R14, R7: 0, Resistors_SMD:R_0603, symbol R
- added R16, R17, R18, R19: 0, Resistors_SMD:R_1206, symbol R
- C10: renamed from C12; footprint (none) -> Capacitors_SMD:C_0603
- C11: renamed from C13; footprint (none) -> Capacitors_SMD:C_0603
- C12: renamed from C14; footprint (none) -> Capacitors_SMD:C_0603
- C13: renamed from C15; footprint (none) -> Capacitors_SMD:C_0603
- C14: renamed from C16; footprint (none) -> Capacitors_SMD:C_0603
- C15: renamed from C17; footprint (none) -> Capacitors_SMD:C_1210
- C16: renamed from C18; footprint (none) -> Capacitors_SMD:C_0603
- C17: renamed from C20; footprint (none) -> Capacitors_SMD:C_0603
- C18: renamed from C21; footprint (none) -> Capacitors_SMD:C_0603
- C19: renamed from C22; footprint (none) -> Capacitors_SMD:C_0603
- C20: renamed from C23; footprint (none) -> Capacitors_SMD:C_0603
- C21: renamed from C24; footprint (none) -> Capacitors_SMD:C_0603
- C22: renamed from C25; footprint (none) -> Capacitors_SMD:C_0603
- C23: renamed from C27; footprint (none) -> Capacitors_SMD:C_0603
- C24: renamed from C28; footprint (none) -> Capacitors_SMD:C_0603
- C25: renamed from C29; footprint (none) -> Capacitors_SMD:C_0603
- C26: renamed from C30; footprint (none) -> Capacitors_SMD:C_0603
- C27: renamed from C31; footprint (none) -> Capacitors_SMD:C_0603
- C28: renamed from C32; footprint (none) -> Capacitors_SMD:C_0603
- C3: footprint (none) -> Capacitors_SMD:C_0603
- C4: footprint (none) -> Capacitors_SMD:C_1210
- C5: renamed from C6; footprint (none) -> Capacitors_SMD:C_0603
- C6: renamed from C7; footprint (none) -> Capacitors_SMD:C_0603
- C7: renamed from C8; footprint (none) -> Capacitors_SMD:C_0603
- C8: renamed from C9; footprint (none) -> Capacitors_SMD:C_0603
- C9: renamed from C11; footprint (none) -> Capacitors_SMD:C_0603
- R1, R10, R11, R12, R15, R2, R3, R4, R8, R9: footprint (none) -> Resistors_SMD:R_0603
- R13, R6: value 15k8 -> 5k9; footprint (none) -> Resistors_SMD:R_0603
- R5: footprint (none) -> Resistors_SMD:R_1206
- U1, U5: footprint (none) -> Housings_SSOP:TSSOP-8_3x3mm_Pitch0.65mm
- U10, U3, U7, U8, U9: footprint TO_SOT_Packages_SMD:SOT-23-5 -> TO-220-5:TO-220-5_Pentawatt_Multiwatt-5_Vertical_StaggeredType1
- U2, U6: footprint (none) -> Housings_SOIC:SOIC-8_3.9x4.9mm_Pitch1.27mm
Connections:
- net GNDA: now also J18.1
- net Iin: now also J7.1
- net Iout: now also J12.1
- net Vin: now also J13.1
- net Vout: now also J17.1, R16.2, R17.2, R18.2, R19.2; no longer U10.5, U7.5, U8.5, U9.5
- net at C4.2, R4.1, U1.3 (+): now also J8.1
- net at R1.1, R2.1, U1.1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: now also J9.1
- net at R8.1, U1.6 (-): now also R6.2
- net at C3.1, R1.2, R6.1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: now also J10.1, R7.2; no longer U1.7
- net at R5.1, U2.2, U3.5: now also J11.1
- net at C15.2, R12.1, U5.3 (+): now also J14.1
- net at R10.1, R9.1, U5.1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: now also J15.1
- net at C14.1, R13.1, R9.2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: now also J16.1, R14.2; no longer U5.7
- net at R13.2: now also R15.1, U5.6 (-)
- new net: R7.1, U1.7
- new net: R16.1, U7.5
- new net: R17.1, U8.5
- new net: R18.1, U9.5
- new net: R19.1, U10.5
- new net: R14.1, U5.7
Other:
- note added: "2-pole 100kHz LP Butterworth\nTAOE3 Sallen and Key 6.3.2"
- note added: "2-pole 100kHz LP Butterworth\nTAOE3 Salllen and Key 6.3.2"
- note added: "DC block"
- note added: "LT1010 DS parallel operation"
- note added: "TAOE3 5.14.2D current sources"
- note removed: "100 Ohm"
- note removed: "2-pole Butterworth"
- moved on the sheet: R13, R15, R6, R8
